Commit message: Update ros2_ws: Configure ros2 controllers and debug with HW interface and gazebo sim, Create a custom controller

File: src/dobo_description/urdf/mobile_base.ros2_control.xacro (robot description, xacro)
@@ -1,8 +1,14 @@
 <?xml version="1.0"?>
 <robot name="my_robot" xmlns:xacro="http://www.ros.org/wiki/xacro">
-  <ros2_control name="MobileBaseHardwareInterface" type="system">
+  <ros2_control name="MobileBase" type="system">
     <hardware>
-      <plugin>mock_components/GenericSystem</plugin>
+     <plugin>mock_components/GenericSystem</plugin>
       <param name="calculate_dynamics">true</param>
+<!--
+      <plugin>mobile_base_hardware/MobileBaseHardwareInterface</plugin>
+      <param name="left_motor_id">10</param>
+      <param name="right_mrotor_id">20</param>
+      <param name="port">/dev/ttyACM0</param>
+-->
     </hardware>
     <joint name="base_left_wheel_joint">

File: src/dobo_description/urdf/my_robot.urdf.xacro (robot description, xacro)
@@ -4,4 +4,11 @@
     <xacro:include filename="mobile_base.xacro" />
     <xacro:include filename="mobile_base.ros2_control.xacro" />
+    <xacro:include filename="arm.xacro" />
+    <joint name="mobile_base_arm_joint" type="fixed">
+        <parent link="base_link" />
+        <child link="arm_base_link"/>
+        <origin xyz="${base_length /3.0} 0 ${base_heigth}" rpy="0 0 0" />
+    </joint>
+  <xacro:include filename="arm.ros2_control.xacro" />
   <!--
     <xacro:include filename="mobile_base_gazebo.xacro" />
