Commit message: Update ros2_ws: Control robot arm with Moveit and using Cpp API

File: src/robot_arm_description/urdf/common_properties.xacro (robot description, xacro)
@@ -13,3 +13,9 @@
         <color rgba="0 0 0.5 1"/>
     </material>
+    <material name="dark_green">
+        <color rgba="0 0.4 0 1" />
+    </material>
+    <material name="light_green">
+        <color rgba="0 0.6 0 1" />
+    </material>
 </robot>

File: src/robot_arm_description/urdf/my_arm.ros2_control.xacro (robot description, xacro)
@@ -1,7 +1,5 @@
 <?xml version="1.0"?>
 <robot xmlns:xacro="http://www.ros.org/wiki/xacro">
-    <xacro:macro name="my_arm_ros2_control" params="name initial_positions_file">
-        <xacro:property name="initial_positions" value="${xacro.load_yaml(initial_positions_file)['initial_positions']}"/>
-        <ros2_control name="${name}" type="system">
+        <ros2_control name="Arm" type="system">
             <hardware>
                 <!-- By default, set up controllers for simulation. This won't work on real hardware -->
@@ -11,5 +9,5 @@
                 <command_interface name="position"/>
                 <state_interface name="position">
-                  <param name="initial_value">${initial_positions['joint1']}</param>
+                  <param name="initial_value">0.0</param>
                 </state_interface>
             </joint>
@@ -17,5 +15,5 @@
                 <command_interface name="position"/>
                 <state_interface name="position">
-                  <param name="initial_value">${initial_positions['joint2']}</param>
+                  <param name="initial_value">0.0</param>
                 </state_interface>
             </joint>
@@ -23,5 +21,5 @@
                 <command_interface name="position"/>
                 <state_interface name="position">
-                  <param name="initial_value">${initial_positions['joint3']}</param>
+                  <param name="initial_value">0.0</param>
                 </state_interface>
             </joint>
@@ -29,5 +27,5 @@
                 <command_interface name="position"/>
                 <state_interface name="position">
-                  <param name="initial_value">${initial_positions['joint4']}</param>
+                  <param name="initial_value">0.0</param>
                 </state_interface>
             </joint>
@@ -35,5 +33,5 @@
                 <command_interface name="position"/>
                 <state_interface name="position">
-                  <param name="initial_value">${initial_positions['joint5']}</param>
+                  <param name="initial_value">0.0</param>
                 </state_interface>
             </joint>
@@ -41,5 +39,5 @@
                 <command_interface name="position"/>
                 <state_interface name="position">
-                  <param name="initial_value">${initial_positions['joint6']}</param>
+                  <param name="initial_value">0.0</param>
                 </state_interface>
             </joint>
@@ -47,8 +45,7 @@
                 <command_interface name="position"/>
                 <state_interface name="position">
-                  <param name="initial_value">${initial_positions['gripper_left_finger_joint']}</param>
+                  <param name="initial_value">0.0</param>
                 </state_interface>
             </joint>
         </ros2_control>
-    </xacro:macro>
 </robot>

File: src/robot_arm_description/urdf/my_arm.urdf.xacro (robot description, xacro)
@@ -3,3 +3,10 @@
     <xacro:include filename="common_properties.xacro" />
     <xacro:include filename="arm.xacro" />
+    <xacro:include filename="gripper.xacro" />
+    <xacro:include filename="my_arm.ros2_control.xacro" />
+    <joint name="gripper_base_joint" type="fixed">
+        <parent link="tool_link" />
+        <child link="gripper_base_link" />
+        <origin xyz="0 0 0" rpy="0 0 0" />
+    </joint>
 </robot>
