Commit message: Update ros2_ws: Control arm with python API an connect with Moveit to hardware

File: src/robot_arm_description/urdf/my_arm.ros2_control.xacro (robot description, xacro)
@@ -1,8 +1,17 @@
 <?xml version="1.0"?>
 <robot xmlns:xacro="http://www.ros.org/wiki/xacro">
+        <xacro:arg name = "use_mock_component" default="true" />
         <ros2_control name="Arm" type="system">
             <hardware>
+              <xacro:if value="$(arg use_mock_component)">
                 <!-- By default, set up controllers for simulation. This won't work on real hardware -->
                 <plugin>mock_components/GenericSystem</plugin>
+              </xacro:if>
+              <xacro:unless value="$(arg use_mock_component)">
+                <plugin>arm_hardware/ArmHardwareInterface</plugin>
+                <param name="joint1_motor_id">10</param>
+                <param name="joint2_motor_id">20</param>
+                <param name="port">/dev/tty/ACM0</param>
+              </xacro:unless>
             </hardware>
             <joint name="joint1">
@@ -42,5 +51,11 @@
                 </state_interface>
             </joint>
-            <joint name="gripper_left_finger_joint">
+        </ros2_control>
+        <ros2_control name="Gripper" type="system">
+            <hardware>
+                <!-- By default, set up controllers for simulation. This won't work on real hardware -->
+                <plugin>mock_components/GenericSystem</plugin>
+          </hardware>
+          <joint name="gripper_left_finger_joint">
                 <command_interface name="position"/>
                 <state_interface name="position">
