Commit message: Update ros2_ws: Create new robot_arm, robot_arm_config_pkg, new_robot_arm_bringup for my custom robot arm.

File: src/robot_arm/urdf/robot_arm.ros2_control.xacro (robot description, xacro)
@@ -1,56 +1,48 @@
 <?xml version="1.0"?>
 <robot xmlns:xacro="http://www.ros.org/wiki/xacro">
-        <xacro:arg name = "use_mock_component" default="true" />
-        <ros2_control name="Arm" type="system">
-            <hardware>
-              <xacro:if value="$(arg use_mock_component)">
-                <!-- By default, set up controllers for simulation. This won't work on real hardware -->
-                <plugin>mock_components/GenericSystem</plugin>
-              </xacro:if>
-              <xacro:unless value="$(arg use_mock_component)">
-                <plugin>arm_hardware/ArmHardwareInterface</plugin>
-                <param name="joint1_motor_id">10</param>
-                <param name="joint2_motor_id">20</param>
-                <param name="port">/dev/tty/ACM0</param>
-              </xacro:unless>
-            </hardware>
-            <joint name="base_rotating_waste_joint">
-                <command_interface name="position"/>
-                <state_interface name="position">
-                  <param name="initial_value">0.0</param>
-                </state_interface>
-            </joint>
-            <joint name="rotating_waste_arm1_joint">
-                <command_interface name="position"/>
-                <state_interface name="position">
-                  <param name="initial_value">0.0</param>
-                </state_interface>
-            </joint>
-            <joint name="arm1_arm2_joint">
-                <command_interface name="position"/>
-                <state_interface name="position">
-                  <param name="initial_value">0.0</param>
-                </state_interface>
-            </joint>
-            <joint name="arm2_gripper_base_joint">
-                <command_interface name="position"/>
-                <state_interface name="position">
-                  <param name="initial_value">0.0</param>
-                </state_interface>
-            </joint>
-        </ros2_control>
-        <ros2_control name="Gripper" type="system">
-            <hardware>
-                <!-- By default, set up controllers for simulation. This won't work on real hardware -->
-                <plugin>mock_components/GenericSystem</plugin>
-                 <!-- <plugin>arduino_arm_hardware::ArduinoArmHardwareInterface</plugin>
-                  <param name="port">/dev/ttyACM0</param> -->
-          </hardware>
-          <joint name="gripper_base_left_gear_joint">
-                <command_interface name="position"/>
-                <state_interface name="position">
-                  <param name="initial_value">0.0</param>
-                </state_interface>
-            </joint>
-        </ros2_control>
+  <!-- Arm system -->
+  <ros2_control name="Arm" type="system">
+    <hardware>
+        <plugin>arduino_arm_hardware::ArduinoArmHardwareInterface</plugin>
+            <param name="port">/dev/ttyACM0</param>
+        <!-- <plugin>mock_components/GenericSystem</plugin> -->
+    </hardware>
+    <!-- Joints -->
+    <joint name="base_rotating_waste_joint">
+      <command_interface name="position"/>
+      <state_interface name="position">
+        <param name="initial_value">0.0</param>
+      </state_interface>
+    </joint>
+    <joint name="rotating_waste_arm1_joint">
+      <command_interface name="position"/>
+      <state_interface name="position">
+        <param name="initial_value">0.0</param>
+      </state_interface>
+    </joint>
+    <joint name="arm1_arm2_joint">
+      <command_interface name="position"/>
+      <state_interface name="position">
+        <param name="initial_value">0.0</param>
+      </state_interface>
+    </joint>
+    <joint name="arm2_gripper_base_joint">
+      <command_interface name="position"/>
+      <state_interface name="position">
+        <param name="initial_value">0.0</param>
+      </state_interface>
+    </joint>
+  </ros2_control>
+  <!-- Gripper system -->
+  <ros2_control name="Gripper" type="system">
+    <hardware>
+        <plugin>mock_components/GenericSystem</plugin>
+         </hardware>
+    <joint name="gripper_base_left_gear_joint">
+      <command_interface name="position"/>
+      <state_interface name="position">
+        <param name="initial_value">0.0</param>
+      </state_interface>
+    </joint>
+  </ros2_control>
 </robot>

File: src/robot_arm/urdf/robot_arm.urdf (robot description, URDF)
Before this commit: robot None, 7 links, 6 joints
Joints:
- joint arm1_arm2_joint: axis -1 0 0 -> 1 0 0; limit lower=-1.57 upper=1.57 effort=300 velocity=2 -> lower=-1.572 upper=1.572 effort=300 velocity=2

File: src/robot_arm/urdf/robot_arm.urdf.xacro (robot description, xacro)
@@ -1,4 +1,4 @@
 <?xml version="1.0"?>
-<robot name="robot_arm" xmlns:xacro="http://www.ros.org/wiki/xacro">
+<robot name="my_arm" xmlns:xacro="http://www.ros.org/wiki/xacro">
     <xacro:include filename="robot_arm.urdf" />
     <xacro:include filename="robot_arm.ros2_control.xacro" />
